File: electrical/pcb/control_board/Control_Boards.kicad_pcb (KiCad board)
At the start: 2 copper layers, 220 x 329.2 mm, 148 parts, among them J1 XT30-M, J10 Molex_172675-0613, J11 Molex_172675-0613, J12 TSW-104-07-F-T, J13 Molex_172675-0613, J14 Molex_172675-0613, J16 277-11404-ND, J17 277-11404-ND, J18 277-11404-ND, J19 TSW-104-07-F-T, J2 ED2580-ND, J20 PEC08SAAN, J21 PPTC102LFBN-RC, J22 S9175-ND_rpi_breakout, J23 S9175-ND_rpi_breakout, J24 6posheader, J25 SSW-104-01-F-T, J26 WM6548-ND, J27 PPTC021LFBN-RC, J28 PPTC021LFBN-RC, J29 PPTC021LFBN-RC, J3 XT30-F, J30 PEC08SAAN, J4 XT30-F, J5 XT30-M, J6 ED2580-ND, J7 TSW-104-07-F-T, J8 Molex_172675-0613, J9 Molex_172675-0613, M1 Mounting_Holes, Q1 2N3906, Q2 2N3906, Q3 2N3906, Q4 2N3906, Q5 2N3906, Q6 2N3906, SW1 CT206124-ND, T1 test_point, T10 test_point, T11 test_point, T12 test_point, T13 test_point, T14 test_point, T15 test_point, T2 test_point, T3 test_point, T4 test_point, T5 test_point, T6 test_point, T7 test_point, T8 test_point, T9 test_point, U1 INA260, U2 PCA9685, U3 D24V22Fx, U4 D24V150Fx, U5 DC7G3HWA, U6 DC7G3HWA, U7 MIC2937A-3.3WT, y1 rover_silkscreen, y2 rover_silkscreen

Commit message: Control board - document v203, remove old (#560)
* update to kicad10, bump rev on back of motor board to v2.0.3

* generate 3d_images for v2.0.3, and add script to automate that process

* added scripts to export layout documentation, and v2.0.3 layout files.

* updated 3d_images exports and scripts to adjust bounding box calculations.  Moved documentation scripts to documentation/utilities

* moved documentation utilities to new dir.

* update schematics to kicad 10, add titles and versions to title blocks

* updated export_schematic script to expand ${VERSION} properly, plus new schematics and 3d_images

* add gerbers for v2.0.3, and export script

* Remove old control board revs.  Based on discussion in https://github.com/nasa-jpl/open-source-rover/issues/444, remove documentation of old versions of control boards.

* Remove more old control board revs, reorg images.

* Remove more old control board revs, reorg images.

* Fix figure cross-references and normalize "Figure" capitalization

Inserting "Figure 3.17: INA260 bypassed" shifted every later section-3
caption by one, but the renumbering pass only matched capital-F "Figure".
The 17 lowercase "figure N.N" prose references were left behind, so nine
of them pointed one figure short of their subject -- e.g. the 3.3V
regulator direction cited "U7 footprint" rather than the photo of the
regulator installed in U7.

Repoints those nine at the captions they describe, verified by matching
each reference against the caption text at 83fcd96 (before the shift):

  3.23 -> 3.24  3.3V regulator orientation
  3.24 -> 3.25  C7 polarity
  3.32 -> 3.33  headers in the U2 footprint
  3.33 -> 3.34  male headers on the PCA9685
  3.34 -> 3.35  1x1 pin/header option
  3.39 -> 3.40  RC2 capacitors
  3.40 -> 3.41  RC1 and RC3 capacitors
  3.42 -> 3.43  roboclaw terminal block wiring

Also capitalizes all 17 lowercase references to "Figure" so prose matches
the caption spelling. Every figure reference in the file now resolves to
an ex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
Other:
- board text added: "Open Source Rover Robotic Breakout Boards - Brain Board - ${VERSION}"
- board text added: "Open Source Rover Robotic Breakout Boards Brain Board ${VERSION}"
- board text added: "Open Source Rover Robotic Breakout Boards Motor Board - ${VERSION}"
- board text removed: "Open Source Rover Robotic Breakout Boards - Brain Board - v2.0.3"
- board text removed: "Open Source Rover Robotic Breakout Boards Brain Board v2.0.2"
- board text removed: "Open Source Rover Robotic Breakout Boards Motor Board - v2.0.3"
